File: pcb/esphome-humitemp.kicad_pcb (KiCad board)
At the start: 2 copper layers, 45 x 30 mm, 18 parts, among them J2 USB_IN, SW1 RESET, U1 SHT3x, U3 AMS1117-3.3, U4 ESP32-C3-MINI-1

Commit message: fix a few issues
Parts:
- removed H4: MountingHole, MountingHole:MountingHole_3.2mm_M3
Changed lines of the file:
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@@
     )
-  )
-  (footprint "MountingHole:MountingHole_3.2mm_M3" (layer "F.Cu")
-    (at 100 36)
-    (descr "Mounting Hole 3.2mm, no annular, M3")
-    (tags "mounting hole 3.2mm no annular m3")
-    (property "Sheetfile" "esphome-humitemp.kicad_sch")
-    (property "Sheetname" "")
-    (property "ki_description" "Mounting Hole without connection")
-    (property "ki_keywords" "mounting hole")
-    (solder_mask_margin 1.9)
-    (clearance 2)
-    (attr exclude_from_pos_files)
-    (fp_text reference "H4" (at 0 -4.2) (layer "F.SilkS") hide
-        (effects (font (size 1 1) (thickness 0.15)))
-    )
-    (fp_text value "MountingHole" (at 0 4.2) (layer "F.Fab")
-        (effects (font (size 1 1) (thickness 0.15)))
-    )
-    (fp_text user "${REFERENCE}" (at 0.3 0) (layer "F.Fab")
-        (effects (font (size 1 1) (thickness 0.15)))
-    )
-    (fp_circle (center 0 0) (end 3.2 0)
-      (stroke (width 0.15) (type solid)) (fill none) (layer "Cmts.User"))
-    (fp_circle (center 0 0) (end 3.45 0)
-      (stroke (width 0.05) (type solid)) (fill none) (layer "F.CrtYd"))
-    (pad "" np_thru_hole circle (at 0 0) (size 3.2 3.2) (drill 3.2) (layers "*.Cu" "*.Mask"))
   )
   (footprint "Capacitor_SMD:C_0603_1608Metric" (layer "F.Cu")
