File: pcb/esphome-humitemp.kicad_sch (KiCad schematic)
At the start: 19 parts, among them J2 USB_IN, SW1 RESET, U1 SHT3x, U3 AMS1117-3.3, U4 ESP32-C3-MINI-1

Commit message: fix a few issues
Parts:
- removed H3, H4: MountingHole, MountingHole:MountingHole_3.2mm_M3, symbol Mechanical:MountingHole
Changed lines of the file:
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@@
-    )
-  )
-  (symbol (lib_id "Mechanical:MountingHole") (at 20.32 147.32 0) (unit 1)
-    (in_bom yes) (on_board yes) (dnp no) (fields_autoplaced)
-    (property "Reference" "H4" (at 24.13 146.0499 0)
-      (effects (font (size 1.27 1.27)) (justify left))
-    )
-    (property "Value" "MountingHole" (at 24.13 148.5899 0)
-      (effects (font (size 1.27 1.27)) (justify left))
-    )
-    (property "Footprint" "MountingHole:MountingHole_3.2mm_M3" (at 20.32 147.32 0)
-      (effects (font (size 1.27 1.27)) hide)
-    )
-    (property "Datasheet" "~" (at 20.32 147.32 0)
-      (effects (font (size 1.27 1.27)) hide)
-    )
-    (instances
-      (project "esphome-humitemp"
-        (path "/9ed555b5-b872-4c07-8527-e7d67b145785"
-          (reference "H4") (unit 1)
-        )
-      )
     )
   )
@@
         )
       )
-    )
-  )
-  (symbol (lib_id "Mechanical:MountingHole") (at 20.32 142.24 0) (unit 1)
-    (in_bom yes) (on_board yes) (dnp no) (fields_autoplaced)
-    (property "Reference" "H3" (at 24.13 140.9699 0)
-      (effects (font (size 1.27 1.27)) (justify left))
-    )
-    (property "Value" "MountingHole" (at 24.13 143.5099 0)
-      (effects (font (size 1.27 1.27)) (justify left))
-    )
-    (property "Footprint" "MountingHole:MountingHole_3.2mm_M3" (at 20.32 142.24 0)
-      (effects (font (size 1.27 1.27)) hide)
-    )
-    (property "Datasheet" "~" (at 20.32 142.24 0)
-      (effects (font (size 1.27 1.27)) hide)
-    )
-    (instances
-      (project "esphome-humitemp"
-        (path "/9ed555b5-b872-4c07-8527-e7d67b145785"
-          (reference "H3") (unit 1)
-        )
-      )

Commit message: fix part number for 10k
Parts:
- R2, R3: LCSC C17414 -> C25744
Changed lines of the file:
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@@
       (effects (font (size 1.27 1.27)) hide)
     )
-    (property "LCSC" "C17414" (at 49.53 69.85 0)
+    (property "LCSC" "C25744" (at 49.53 69.85 0)
       (effects (font (size 1.27 1.27)) hide)
     )
@@
       (effects (font (size 1.27 1.27)) hide)
     )
-    (property "LCSC" "C17414" (at 58.42 72.39 0)
+    (property "LCSC" "C25744" (at 58.42 72.39 0)
       (effects (font (size 1.27 1.27)) hide)
     )
